File: Hardware/digital-clock-ne555.kicad_pcb (KiCad board)
At the start: 2 copper layers, 100 x 90 mm, 59 parts, among them J1 CONN_01X02, SW1 SW_Push, SW2 SW_Push, SW3 SW_Push, U1 NE555, U10 7SEGMENT_CA, U11 74LS90, U12 74LS47, U13 7SEGMENT_CA, U14 74LS90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

Commit message: unrouted net
Parts:
- removed the ? at (88.5, 120.8)
- added ?: SolderWirePad_single_0-8mmDrill, Wire_Pads:SolderWirePad_single_0-8mmDrill, F.Cu at (120.0, 92.5)
- added ?: SolderWirePad_single_0-8mmDrill, Wire_Pads:SolderWirePad_single_0-8mmDrill, F.Cu at (82.0, 103.0)
- added ?: SolderWirePad_single_0-8mmDrill, Wire_Pads:SolderWirePad_single_0-8mmDrill, F.Cu at (72.5, 108.5)
- added ?: SolderWirePad_single_0-8mmDrill, Wire_Pads:SolderWirePad_single_0-8mmDrill, F.Cu at (120.0, 109.5)
- moved ? 21.9 mm to (120.5, 102.5)
- moved ? 21.6 mm to (110.8, 101.5)
- moved ? 21.6 mm to (60.0, 129.0)
- moved ? 21.6 mm to (57.5, 129.0)
- moved ? 21.6 mm to (55.0, 129.0)
- moved ? 21.6 mm to (144.0, 57.0)
- moved ? 21.6 mm to (144.0, 54.5)
- moved ? 21.6 mm to (144.0, 52.0)
- moved ? 21.6 mm to (134.0, 59.5)
- moved ? 21.6 mm to (118.5, 57.0)
- moved ? 21.6 mm to (106.0, 58.0)
- moved ? 21.6 mm to (65.5, 89.5)
- moved ? 21.6 mm to (88.0, 66.5)
- moved ? 21.6 mm to (98.0, 58.0)
- moved ? 21.6 mm to (86.0, 56.5)
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Routing:
- net /Net7: track 45.5 -> 80.9 mm
- net /Net20: track 0.00 -> 29.0 mm
- net /Net11: track 105.7 -> 102.8 mm
- net Net-(U6-Pad15): track 54.4 -> 56.6 mm
- net /Net17: track 35.6 -> 34.4 mm
- net /Net3: track 30.4 -> 29.4 mm
- net Net-(U18-Pad12): track 36.7 -> 37.6 mm
- net Net-(U18-Pad13): track 42.4 -> 43.1 mm
- net Net-(U6-Pad13): track 42.0 -> 42.6 mm
- net /Net19: track 116.7 -> 116.1 mm
- net Net-(U6-Pad14): track 53.6 -> 53.1 mm
